File: board.sch (KiCad schematic (older format))
At the start: 12 parts, among them J1 PMW3360, J2 MCU, U1 TLV70019_SOT23-5

Commit message: Mounting holes
Parts:
- added J3, J4, J5, J6: Mounting_Hole, MountingHole:MountingHole_2.2mm_M2_Pad_Via, symbol Connector:Conn_01x01_Female
Connections:
- wire segments 62 -> 63
Changed lines of the file:
@@
 L power:+3.3V #PWR0107
 U 1 1 5B2AAC2B
-P 7300 2525
-F 0 "#PWR0107" H 7300 2375 50  0001 C CNN
-F 1 "+3.3V" H 7450 2600 50  0000 C CNN
-F 2 "" H 7300 2525 50  0001 C CNN
-F 3 "" H 7300 2525 50  0001 C CNN
-	1    7300 2525
+P 7750 2400
+F 0 "#PWR0107" H 7750 2250 50  0001 C CNN
+F 1 "+3.3V" H 7900 2475 50  0000 C CNN
+F 2 "" H 7750 2400 50  0001 C CNN
+F 3 "" H 7750 2400 50  0001 C CNN
+	1    7750 2400
 	1    0    0    -1
 $EndComp
@@
 	6925 3100 7750 3100
 Wire Wire Line
-	7300 2525 7300 2600
-Wire Wire Line
 	7300 2925 7225 2925
 Wire Wire Line
-	7725 2750 7725 2600
+	7300 2925 7300 2550
 Wire Wire Line
-	7725 2600 7300 2600
-Connection ~ 7300 2600
+	7300 2550 7750 2550
 Wire Wire Line
-	7300 2600 7300 2925
+	7750 2550 7750 2400
+Wire Wire Line
+	7750 2550 7750 2750
+Wire Wire Line
+	7750 2750 7725 2750
+Connection ~ 7750 2550
+$Comp
+L Connector:Conn_01x01_Female J3
+U 1 1 5B295FD5
+P 6775 650
+F 0 "J3" H 6850 700 50  0000 L CNN
+F 1 "Mounting_Hole" H 6850 625 50  0000 L CNN
+F 2 "MountingHole:MountingHole_2.2mm_M2_Pad_Via" H 6775 650 50  0001 C CNN
+F 3 "~" H 6775 650 50  0001 C CNN
+	1    6775 650
+	1    0    0    -1
+$EndComp
+$Comp
+L Connector:Conn_01x01_Female J4
+U 1 1 5B29617E
+P 6775 800
+F 0 "J4" H 6850 850 50  0000 L CNN
+F 1 "Mounting_Hole" H 6850 775 50  0000 L CNN
+F 2 "MountingHole:MountingHole_2.2mm_M2_Pad_Via" H 6775 800 50  0001 C CNN
+F 3 "~" H 6775 800 50  0001 C CNN
+	1    6775 800
+	1    0    0    -1
+$EndComp
+$Comp
+L Connector:Conn_01x01_Female J5
+U 1 1 5B2961E6
+P 6775 950
+F 0 "J5" H 6850 1000 50  0000 L CNN
+F 1 "Mounting_Hole" H 6850 925 50  0000 L CNN
+F 2 "MountingHole:MountingHole_2.2mm_M2_Pad_Via" H 6775 950 50  0001 C CNN
+F 3 "~" H 6775 950 50  0001 C CNN
+	1    6775 950
+	1    0    0    -1
+$EndComp
+$Comp
+L Connector:Conn_01x01_Female J6
+U 1 1 5B29621C
+P 6775 1100
+F 0 "J6" H 6850 1150 50  0000 L CNN
+F 1 "Mounting_Hole" H 6850 1075 50  0000 L CNN
+F 2 "MountingHole:MountingHole_2.2mm_M2_Pad_Via" H 6775 1100 50  0001 C CNN
+F 3 "~" H 6775 1100 50  0001 C CNN
+	1    6775 1100
+	1    0    0    -1
+$EndComp
 $EndSCHEMATC

Commit message: Add manf#
Parts:
- C1: manf# (none) -> MCTT21F475Z100CT
- C2: manf# (none) -> 0805B104K500CT
- C3, C4: manf# (none) -> 0805B105K100CT
- J2: manf# (none) -> 68000-107HLF
- R1, R3, R5: manf# (none) -> MCWR08X1002FTL
- R2: manf# (none) -> MCWR08X39R0FTL
- R4: manf# (none) -> MCWR08X1300FTL
- U1: manf# (none) -> TLV70019DDCT
Changed lines of the file:
@@
 F 1 "PMW3360" H 5900 2500 50  0000 C CNN
 F 2 "Pixart:PMW3360DM-T2QU" H 5850 3000 50  0001 C CNN
-F 3 "~" H 5850 3000 50  0001 C CNN
+F 3 "http://www.pixart.com.tw/upload/PMS0058-PMW3360DM-T2QU-NNDS-R1.30-06042016_20160902201411.pdf" H 5850 3000 50  0001 C CNN
 	1    5850 3000
 	1    0    0    -1
@@
 F 2 "Capacitor_SMD:C_0805_2012Metric" H 4338 1875 50  0001 C CNN
 F 3 "~" H 4300 2025 50  0001 C CNN
+F 4 "MCTT21F475Z100CT" H 4300 2025 50  0001 C CNN "manf#"
 	1    4300 2025
 	1    0    0    -1
@@
 F 2 "Capacitor_SMD:C_0805_2012Metric" H 4888 1875 50  0001 C CNN
 F 3 "~" H 4850 2025 50  0001 C CNN
+F 4 "0805B104K500CT" H 4850 2025 50  0001 C CNN "manf#"
 	1    4850 2025
 	1    0    0    -1
@@
 F 2 "Resistor_SMD:R_0805_2012Metric" V 6580 2800 50  0001 C CNN
 F 3 "~" H 6650 2800 50  0001 C CNN
+F 4 "MCWR08X39R0FTL" H 6650 2800 50  0001 C CNN "manf#"
 	1    6650 2800
 	0    -1   -1   0
@@
 F 2 "Resistor_SMD:R_0805_2012Metric" V 5080 3300 50  0001 C CNN
 F 3 "~" H 5150 3300 50  0001 C CNN
+F 4 "MCWR08X1002FTL" H 5150 3300 50  0001 C CNN "manf#"
 	1    5150 3300
 	0    -1   -1   0
@@
 F 2 "Resistor_SMD:R_0805_2012Metric" V 6580 3100 50  0001 C CNN
 F 3 "~" H 6650 3100 50  0001 C CNN
+F 4 "MCWR08X1300FTL" H 6650 3100 50  0001 C CNN "manf#"
 	1    6650 3100
 	0    -1   -1   0
@@
 F 2 "Package_TO_SOT_SMD:SOT-23-5" H 9325 1425 50  0001 C CIN
 F 3 "http://www.ti.com/lit/ds/symlink/tlv700.pdf" H 9325 1150 50  0001 C CNN
+F 4 "TLV70019DDCT" H 9325 1100 50  0001 C CNN "manf#"
 	1    9325 1100
 	1    0    0    -1
@@
 F 2 "Capacitor_SMD:C_0805_2012Metric" H 9863 1050 50  0001 C CNN
 F 3 "~" H 9825 1200 50  0001 C CNN
+F 4 "0805B105K100CT" H 9825 1200 50  0001 C CNN "manf#"
 	1    9825 1200
 	1    0    0    -1
@@
 F 2 "Capacitor_SMD:C_0805_2012Metric" H 8738 1000 50  0001 C CNN
 F 3 "~" H 8700 1150 50  0001 C CNN
+F 4 "0805B105K100CT" H 8700 1150 50  0001 C CNN "manf#"
 	1    8700 1150
 	1    0    0    -1
@@
 F 2 "Connector_PinHeader_2.54mm:PinHeader_1x07_P2.54mm_Vertical" H 7950 3300 50  0001 C CNN
 F 3 "~" H 7950 3300 50  0001 C CNN
+F 4 "68000-107HLF" H 7950 3300 50  0001 C CNN "manf#"
 	1    7950 3300
 	1    0    0    -1
@@
 F 2 "Resistor_SMD:R_0805_2012Metric" V 7505 2750 50  0001 C CNN
 F 3 "~" H 7575 2750 50  0001 C CNN
+F 4 "MCWR08X1002FTL" H 7575 2750 50  0001 C CNN "manf#"
 	1    7575 2750
 	0    -1   -1   0
@@
 F 2 "Resistor_SMD:R_0805_2012Metric" V 7005 2925 50  0001 C CNN
 F 3 "~" H 7075 2925 50  0001 C CNN
+F 4 "MCWR08X1002FTL" H 7075 2925 50  0001 C CNN "manf#"
 	1    7075 2925
 	0    -1   -1   0
